File: esc/power.kicad_sch (KiCad schematic)
At the start: 16 parts

Commit message: with phase
Parts:
- added D2: LED, symbol Device:LED
- added R8: 1k, symbol Device:R
Connections:
- net 3V3: now also D2.2 (A)
- net GND: now also R8.2
- net BUCK_FB: now reaches R5.2, R6.1, TP6841S6.3 (FB)
- net BUCK_VIN: now reaches C12.1, C9.1, FB1.2, R3.1, TP6841S6.5 (VIN)
- net BUCK_EN: now reaches R3.2, R4.1, TP6841S6.4 (EN)
- net BUCK_BST: now reaches C13.1, TP6841S6.1 (BST)
- net BUCK_SW: now reaches C13.2, L1.1, TP6841S6.6 (SW)
- new net LED_PWR_K: D2.1 (K), R8.1
Other:
- note added: "V_EN = 1.2V Vcc_low = 10.8V"
- moved on the sheet: C10, C11, C12, C13, C14, C9, D1, FB1, L1, R1, R2, R3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
