File: esc/amplify.kicad_sch (KiCad schematic)
At the start: 13 parts, among them IC2 AD8221ARMZ

Commit message: adding esc kicad and stm32cubeide project
Parts:
- R24, R25: Link https://www.mouser.de/ProductDetail/Panasonic/ERA-1AEB103C?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 -> https://www.mouser.de/ProductDetail/SEI-Stackpole/RNCE0603B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; MF Panasonic -> SEI Stackpole; MP ERA-1AEB103C -> RNCE0603BTE10K0; MPN 667-ERA-1AEB103C -> 708-RNCE0603BTE10K0
Changed lines of the file:
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@@
 			)
 		)
-		(property "Link" "https://www.mouser.de/ProductDetail/Panasonic/ERA-1AEB103C?qs=6%252Bc%252B2ke79U4Rqou4jG9qiw%3D%3D"
-			(at 177.8 115.57 0)
-			(effects
-				(font
-					(size 1.27 1.27)
-				)
-				(hide yes)
-			)
-		)
-		(property "MF" " Panasonic "
-			(at 177.8 115.57 0)
-			(effects
-				(font
-					(size 1.27 1.27)
-				)
-				(hide yes)
-			)
-		)
-		(property "MP" "ERA-1AEB103C "
-			(at 177.8 115.57 0)
-			(effects
-				(font
-					(size 1.27 1.27)
-				)
-				(hide yes)
-			)
-		)
-		(property "MPN" "667-ERA-1AEB103C "
+		(property "Link" "https://www.mouser.de/ProductDetail/SEI-Stackpole/RNCE0603BTE10K0?qs=efUn273yAhfamz7JFGXL1Q%3D%3D"
+			(at 177.8 115.57 0)
+			(effects
+				(font
+					(size 1.27 1.27)
+				)
+				(hide yes)
+			)
+		)
+		(property "MF" "SEI Stackpole "
+			(at 177.8 115.57 0)
+			(effects
+				(font
+					(size 1.27 1.27)
+				)
+				(hide yes)
+			)
+		)
+		(property "MP" "RNCE0603BTE10K0 "
+			(at 177.8 115.57 0)
+			(effects
+				(font
+					(size 1.27 1.27)
+				)
+				(hide yes)
+			)
+		)
+		(property "MPN" "708-RNCE0603BTE10K0 "
 			(at 177.8 115.57 0)
 			(effects
@@
 			)
 		)
-		(property "Link" "https://www.mouser.de/ProductDetail/Panasonic/ERA-1AEB103C?qs=6%252Bc%252B2ke79U4Rqou4jG9qiw%3D%3D"
-			(at 177.8 107.95 0)
-			(effects
-				(font
-					(size 1.27 1.27)
-				)
-				(hide yes)
-			)
-		)
-		(property "MF" " Panasonic "
-			(at 177.8 107.95 0)
-			(effects
-				(font
-					(size 1.27 1.27)
-				)
-				(hide yes)
-			)
-		)
-		(property "MP" "ERA-1AEB103C "
-			(at 177.8 107.95 0)
-			(effects
-				(font
-					(size 1.27 1.27)
-				)
-				(hide yes)
-			)
-		)
-		(property "MPN" "667-ERA-1AEB103C "
-			(at 177.8 107.95 0)
-			(effects
+		(property "Link" "https://www.mouser.de/ProductDetail/SEI-Stackpole/RNCE0603BTE10K0?qs=efUn273yAhfamz7JFGXL1Q%3D%3D"
+			(at 177.8 107.95 0)
+			(effects
+				(font
+					(size 1.27 1.27)
+				)
+				(hide yes)
+			)
+		)
+		(property "MF" "SEI Stackpole "
+			(at 177.8 107.95 0)
+			(effects
+				(font
+					(size 1.27 1.27)
+				)
+				(hide yes)
+			)
+		)
+		(property "MP" "RNCE0603BTE10K0 "
+			(at 177.8 107.95 0)
+			(effects
+				(font
+					(size 1.27 1.27)
+				)
+				(hide yes)
+			)
+		)
+		(property "MPN" "708-RNCE0603BTE10K0 "
+			(at 177.8 107.95 0)
+			(effects
