File: esc/phase.kicad_sch (KiCad schematic)
At the start: 17 parts, among them IC1 IR2103STRPBF, IC2 INA180A3IDBVT, Q1 SiR182DP-T1-RE3, Q2 SiR182DP-T1-RE3

Commit message: esc changes
Parts:
- added C34: 1u, symbol Device:C
Connections:
- net VB: now also C34.1
- net VPH: now also C34.2
- net VLO: now reaches IC1.5 (LO), R12.2
Other:
- note added: "Amplifier to measure voltage drop"

Commit message: full layout
Parts:
- removed D4: 1N5819WS, SamacSys_Parts:SMBJ18A, symbol SamacSys_Parts:SMBJ18A
- removed D5: SMBJ18A, SamacSys_Parts:SMBJ18A, symbol SamacSys_Parts:SMBJ18A
- removed IC1: IR2103STRPBF, SOIC127P600X175-8N, symbol SamacSys_Parts:IR2103STRPBF
- removed IC2: INA180A3IDBVT, SOT95P280X145-5N, symbol SamacSys_Parts:INA180A3IDBVT
- added D10, D5: SMBJ18A-13-F, SamacSys_Parts:DIOM5336X250N, symbol SamacSys_Parts:SMBJ18A-13-F
- added IC3: IR2103STRPBF, SamacSys_Parts:SOIC127P600X175-8N, symbol SamacSys_Parts:IR2103STRPBF
- added IC4: INA180A3IDBVT, SamacSys_Parts:SOT95P280X145-5N, symbol SamacSys_Parts:INA180A3IDBVT
- C28: renamed from C6; footprint (none) -> Capacitor_SMD:C_0603_1608Metric; Link (none) -> https://www.mouser.de/ProductDetail/TAIYO-YUDEN/MBJCT168CB7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; MF (none) -> TAIYO YUDEN; MP (none) -> MBJCT168CB7105KRPA01; MPN (none) -> 963-BJCT168CB7105KR
- C29: renamed from C34; footprint (none) -> Capacitor_SMD:C_0603_1608Metric; Link (none) -> https://www.mouser.de/ProductDetail/TAIYO-YUDEN/MBJCT168CB7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; MF (none) -> TAIYO YUDEN; MP (none) -> MBJCT168CB7105KRPA01; MPN (none) -> 963-BJCT168CB7105KR
- C30: renamed from C20; footprint (none) -> Capacitor_SMD:C_1206_3216Metric; Link (none) -> https://www.mouser.de/ProductDetail/TDK/C3216X5R1E476M160AC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; MF (none) -> TDK; MP (none) -> C3216X5R1E476M160AC; MPN (none) -> 810-C3216X5R1E476M; Manufacturer_Part_Number (none) -> MLASE31LBB5476MTNA01; Mouser Part Number (none) -> 963-MLASE31LBB5476MT
- C31: renamed from C23; footprint (none) -> Capacitor_SMD:C_0402_1005Metric; Link (none) -> https://www.mouser.de/ProductDetail/Vishay-Vitramon/VJ0402Y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; MF (none) -> Vishay / Vitramon; MP (none) -> VJ0402Y103KXJAC31X; MPN (none) -> 77-V0402Y103KXJAC31X
- C32: renamed from C21; footprint (none) -> Capacitor_SMD:C_0402_1005Metric; Link (none) -> https://www.mouser.de/ProductDetail/Murata-Electronics/GRM0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; MF (none) -> Murata Electronics; MP (none) -> GRM02YR60G104ME01L; MPN (none) -> 81-GRM02YR60G104ME1L
- C33: renamed from C22; footprint (none) -> Capacitor_SMD:C_0402_1005Metric; Link (none) -> https://www.mouser.de/ProductDetail/TAIYO-YUDEN/MLASE042SB5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; MF (none) -> TAIYO YUDEN; MP (none) -> MLASE042SB5102MWNA01; MPN (none) -> 963-MLASE042SB5102MW
- Q1, Q2: footprint SI7141DPT1GE3 -> SamacSys_Parts:SI7141DPT1GE3; Link (none) -> https://www.mouser.de/ProductDetail/Vishay-Siliconix/SIR182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; MF (none) -> Vishay / Siliconix; MP (none) -> SIR182DP-T1-RE3; MPN (none) -> 78-SIR182DP-T1-RE3
- R26: renamed from R11; footprint (none) -> Resistor_SMD:R_0603_1608Metric; Link (none) -> https://www.mouser.de/ProductDetail/Susumu/RG0603P-101-D-T1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; MF (none) -> Susumu; MP (none) -> RG0603P-101-D-T10; MPN (none) -> 754-RG0603P-101-D
- R27: renamed from R12; footprint (none) -> Resistor_SMD:R_0603_1608Metric; Link (none) -> https://www.mouser.de/ProductDetail/Susumu/RG0603P-101-D-T1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; MF (none) -> Susumu; MP (none) -> RG0603P-101-D-T10; MPN (none) -> 754-RG0603P-101-D
- R28: renamed from R15; footprint (none) -> Resistor_SMD:R_0603_1608Metric; Link (none) -> https://www.mouser.de/ProductDetail/KOA-Speer/RN73H1ETTP470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; MF (none) -> KOA Speer; MP (none) -> RN73H1ETTP4701D25; MPN (none) -> 660-RN73H1ETP4701D25
- R29: renamed from R16; footprint (none) -> Resistor_SMD:R_0603_1608Metric; Link (none) -> https://www.mouser.de/ProductDetail/Vishay-Dale/CRCW06031K0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; MF (none) -> Vishay / Dale; MP (none) -> CRCW06031K00FKED; MPN (none) -> 71-CRCW06031K00FKED
- R30: renamed from R14; footprint (none) -> Resistor_SMD:R_0603_1608Metric; Link (none) -> https://www.mouser.de/ProductDetail/Vishay-Dale/CRCW06031K0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; MF (none) -> Vishay / Dale; MP (none) -> CRCW06031K00FKED; MPN (none) -> 71-CRCW06031K00FKED
- R31: renamed from R13; footprint (none) -> Resistor_SMD:R_1206_3216Metric; Link (none) -> https://www.mouser.de/ProductDetail/YAGEO/PA1206FRF470R002L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; MF (none) -> YAGEO; MP (none) -> PA1206FRF470R002L; MPN (none) -> 603-P1206FRF470R002L
Connections:
- net 3V3: now also IC4.5 (VS)
- net GND: now also D10.2 (A), IC3.4 (COM), IC4.2 (GND)
- net HIN: now also IC3.2 (HIN)
- net LIN: now also IC3.3 (~{LIN})
- net VB: now also D5.1 (K), IC3.8 (VB)
- net VCC: now also D5.2 (A), IC3.1 (VCC)
- net VHO: now also IC3.7 (HO)
- net VIS: now also IC4.4 (OUT)
- net VLO: now also IC3.5 (LO)
- net VPH: now also D10.1 (K), IC3.6 (VS)
- net V_PH_RS: now also IC4.1 (IN+)
- net VHO_R: now reaches Q1.4 (G), R26.2
- net IN-: now reaches R31.2
- net IN-: now also IC4.3 (IN-)

Commit message: ready for production..?
Parts:
- D5: Link (none) -> https://eu.mouser.com/ProductDetail/Diodes-Incorporated/SMB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; MF (none) -> Diodes Incorporated; MP (none) -> SMBJ18A-13-F; MPN (none) -> 621-SMBJ18A-13-F
- IC3: Link (none) -> https://www.mouser.de/ProductDetail/Infineon-Technologies/I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; MF (none) -> Infineon Technologies; MP (none) -> IR2103STRPBF; MPN (none) -> 942-IR2103STRPBF
- IC4: Link (none) -> https://www.mouser.de/ProductDetail/Texas-Instruments/INA18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; MF (none) -> Texas Instruments; MP (none) -> INA180A3IDBVT; MPN (none) -> 595-INA180A3IDBVT
Changed lines of the file:
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@@
+			)
+		)
+		(property "Link" "https://eu.mouser.com/ProductDetail/Diodes-Incorporated/SMBJ18A-13-F?qs=gaDBXWSqsDBisKX%2FYSuPGA%3D%3D"
+			(at 90.17 66.04 0)
+			(effects
+				(font
+					(size 1.27 1.27)
+				)
+				(hide yes)
+			)
+		)
+		(property "MF" " Diodes Incorporated "
+			(at 90.17 66.04 0)
+			(effects
+				(font
+					(size 1.27 1.27)
+				)
+				(hide yes)
+			)
+		)
+		(property "MP" "SMBJ18A-13-F "
+			(at 90.17 66.04 0)
+			(effects
+				(font
+					(size 1.27 1.27)
+				)
+				(hide yes)
+			)
+		)
+		(property "MPN" "621-SMBJ18A-13-F "
+			(at 90.17 66.04 0)
+			(effects
+				(font
+					(size 1.27 1.27)
+				)
+				(hide yes)
 			)
 		)
@@
 			)
 		)
+		(property "Link" "https://www.mouser.de/ProductDetail/Texas-Instruments/INA180A3IDBVT?qs=5aG0NVq1C4yYIoZxdnrAcQ%3D%3D"
+			(at 129.54 124.46 0)
+			(effects
+				(font
+					(size 1.27 1.27)
+				)
+				(hide yes)
+			)
+		)
+		(property "MF" " Texas Instruments "
+			(at 129.54 124.46 0)
+			(effects
+				(font
+					(size 1.27 1.27)
+				)
+				(hide yes)
+			)
+		)
+		(property "MP" "INA180A3IDBVT "
+			(at 129.54 124.46 0)
+			(effects
+				(font
+					(size 1.27 1.27)
+				)
+				(hide yes)
+			)
+		)
+		(property "MPN" " 595-INA180A3IDBVT "
+			(at 129.54 124.46 0)
+			(effects
+				(font
+					(size 1.27 1.27)
+				)
+				(hide yes)
+			)
+		)
 		(pin "3"
 		)
@@
 				(hide yes)
 			)
+		)
+		(property "Link" "https://www.mouser.de/ProductDetail/Infineon-Technologies/IR2103STRPBF?qs=2r01AXMCG3MUNnnJnNllYQ%3D%3D"
+			(at 71.12 87.63 0)
+			(effects
+				(font
+					(size 1.27 1.27)
+				)
+				(hide yes)
+			)
+		)
+		(property "MF" " Infineon Technologies "
+			(at 71.12 87.63 0)
+			(effects
+				(font
+					(size 1.27 1.27)
+				)
+				(hide yes)
+			)
+		)
+		(property "MP" " IR2103STRPBF "
+			(at 71.12 87.63 0)
+			(effects
+				(font
+					(size 1.27 1.27)
+				)
+				(hide yes)
+			)
+		)
+		(property "MPN" "942-IR2103STRPBF "
+			(at 71.12 87.63 0)
+			(effects
+				(font
+					(size 1.27 1.27)
+				)
+				(hide yes)
+			)

Commit message: adding esc kicad and stm32cubeide project
Parts:
- Q1, Q2: value SiR182DP-T1-RE3 -> SIR180DP-T1-RE3; Link https://www.mouser.de/ProductDetail/Vishay-Siliconix/SIR182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 -> https://www.mouser.de/ProductDetail/Vishay-Siliconix/SIR180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; MP SIR182DP-T1-RE3 -> SIR180DP-T1-RE3; MPN 78-SIR182DP-T1-RE3 -> 78-SIR180DP-T1-RE3
- R26, R27: Link https://www.mouser.de/ProductDetail/Susumu/RG0603P-101-D-T1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 -> https://www.mouser.de/ProductDetail/SEI-Stackpole/RNCE0603B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; MF Susumu -> SEI Stackpole; MP RG0603P-101-D-T10 -> RNCE0603BTE100R; MPN 754-RG0603P-101-D -> 708-RNCE0603BTE100R
- R28: Link https://www.mouser.de/ProductDetail/KOA-Speer/RN73H1ETTP470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 -> https://www.mouser.de/ProductDetail/Susumu/RG1608N-472-W-T5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; MF KOA Speer -> Susumu; MP RN73H1ETTP4701D25 -> RG1608N-472-W-T5; MPN 660-RN73H1ETP4701D25 -> 754-RG1608N-472-WT5
Changed lines of the file:
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@@
 			)
 		)
-		(property "Value" "SiR182DP-T1-RE3"
+		(property "Value" "SIR180DP-T1-RE3"
 			(at 142.24 97.79 0)
 			(effects
@@
 			)
 		)
-		(property "Link" "https://www.mouser.de/ProductDetail/Vishay-Siliconix/SIR182DP-T1-RE3?qs=BZBei1rCqCAnM3726exXMw%3D%3D"
+		(property "Link" "https://www.mouser.de/ProductDetail/Vishay-Siliconix/SIR180DP-T1-RE3?qs=lYGu3FyN48fOYZK9fT%252B0jA%3D%3D"
 			(at 129.54 102.87 0)
 			(effects
@@
 			)
 		)
-		(property "MP" "SIR182DP-T1-RE3 "
+		(property "MP" " SIR180DP-T1-RE3 "
 			(at 129.54 102.87 0)
 			(effects
@@
 			)
 		)
-		(property "MPN" "78-SIR182DP-T1-RE3 "
+		(property "MPN" "78-SIR180DP-T1-RE3 "
 			(at 129.54 102.87 0)
 			(effects
@@
 			)
 		)
-		(property "Link" "https://www.mouser.de/ProductDetail/Susumu/RG0603P-101-D-T10?qs=amGC7iS6iy8p2KCMQy1Fkw%3D%3D"
+		(property "Link" "https://www.mouser.de/ProductDetail/SEI-Stackpole/RNCE0603BTE100R?qs=efUn273yAhcgM9EQ1Aecug%3D%3D"
 			(at 106.68 90.17 0)
 			(effects
@@
 			)
 		)
-		(property "MF" " Susumu "
+		(property "MF" " SEI Stackpole "
 			(at 106.68 90.17 0)
 			(effects
@@
 			)
 		)
-		(property "MP" "RG0603P-101-D-T10 "
+		(property "MP" " RNCE0603BTE100R "
 			(at 106.68 90.17 0)
 			(effects
@@
 			)
 		)
-		(property "MPN" "754-RG0603P-101-D "
+		(property "MPN" "708-RNCE0603BTE100R "
 			(at 106.68 90.17 0)
 			(effects
@@
 			)
 		)
-		(property "Link" "https://www.mouser.de/ProductDetail/KOA-Speer/RN73H1ETTP4701D25?qs=9tvNVxbbcEqGYY49eq7YbA%3D%3D"
+		(property "Link" "https://www.mouser.de/ProductDetail/Susumu/RG1608N-472-W-T5?qs=v5GkGT6DDHgtQLxnmBipeQ%3D%3D"
 			(at 201.93 100.33 0)
 			(effects
@@
 			)
 		)
-		(property "MF" "KOA Speer "
+		(property "MF" "Susumu "
 			(at 201.93 100.33 0)
 			(effects
@@
 			)
 		)
-		(property "MP" "RN73H1ETTP4701D25 "
+		(property "MP" " RG1608N-472-W-T5 "
 			(at 201.93 100.33 0)
 			(effects
@@
 			)
 		)
-		(property "MPN" "660-RN73H1ETP4701D25 "
+		(property "MPN" "754-RG1608N-472-WT5 "
 			(at 201.93 100.33 0)
 			(effects
@@
 			)
 		)
-		(property "Link" "https://www.mouser.de/ProductDetail/Susumu/RG0603P-101-D-T10?qs=amGC7iS6iy8p2KCMQy1Fkw%3D%3D"
+		(property "Link" "https://www.mouser.de/ProductDetail/SEI-Stackpole/RNCE0603BTE100R?qs=efUn273yAhcgM9EQ1Aecug%3D%3D"
 			(at 106.68 95.25 0)
 			(effects
@@
 			)
 		)
-		(property "MF" " Susumu "
+		(property "MF" " SEI Stackpole "
 			(at 106.68 95.25 0)
 			(effects
@@
 			)
 		)
-		(property "MP" "RG0603P-101-D-T10 "
+		(property "MP" " RNCE0603BTE100R "
 			(at 106.68 95.25 0)
 			(effects
@@
 			)
 		)
-		(property "MPN" "754-RG0603P-101-D "
+		(property "MPN" "708-RNCE0603BTE100R "
 			(at 106.68 95.25 0)
 			(effects
@@
 			)
 		)
-		(property "Value" "SiR182DP-T1-RE3"
+		(property "Value" "SIR180DP-T1-RE3"
 			(at 142.24 66.04 0)
 			(effects
@@
 			)
 		)
-		(property "Link" "https://www.mouser.de/ProductDetail/Vishay-Siliconix/SIR182DP-T1-RE3?qs=BZBei1rCqCAnM3726exXMw%3D%3D"
+		(property "Link" "https://www.mouser.de/ProductDetail/Vishay-Siliconix/SIR180DP-T1-RE3?qs=lYGu3FyN48fOYZK9fT%252B0jA%3D%3D"
 			(at 129.54 71.12 0)
 			(effects
@@
 			)
 		)
-		(property "MP" "SIR182DP-T1-RE3 "
+		(property "MP" " SIR180DP-T1-RE3 "
 			(at 129.54 71.12 0)
 			(effects
@@
 			)
 		)
-		(property "MPN" "78-SIR182DP-T1-RE3 "
+		(property "MPN" "78-SIR180DP-T1-RE3 "
 			(at 129.54 71.12 0)
 			(effects
