File: esc/esc.kicad_sch (KiCad schematic)
At the start: 14 parts, among them U1 STM32G474RETx, Y1 NX2016SA-24M-EXS00A-CS08891

Commit message: with phase
Parts:
- removed C6: 100n, symbol Device:C
- added C18, C19: 100n, symbol Device:C
- added D3: LED, symbol Device:LED
- added FB2: 120R, symbol Device:FerriteBead
- added R10, R9: 10k, symbol Device:R
- Y1: footprint NX2016SA24MEXS00ACS08891 -> SamacSys_Parts:NX2016SA24MEXS00ACS08891
Connections:
- net 3V3: now also FB2.1, R9.2
- net GND: now also C18.2, C19.2, R10.1
- net VISENSE_C: now reaches U1.10 (PC2)
- net VISENSE_A: now reaches U1.12 (PA0)
- net VISENSE_B: now reaches U1.14 (PA2)
- net at U1.2 (PC13): now also D3.2 (A)
- net I2C_SCL: now reaches U1.40 (PC8)
- net I2C_SCA: now reaches U1.41 (PC9)
- net HIN_A: now reaches U1.42 (PA8)
- net HIN_B: now reaches U1.43 (PA9)
- net HIN_C: now reaches U1.44 (PA10)
- net at U1.7 (PG10): now also C19.1, R9.1
- new net: D3.1 (K), R10.2
- new net: C18.1, FB2.2
Other:
- added sheet Phase (phase.kicad_sch)
- moved on the sheet: C1, C15, C16, C17, C2, C3, C4, C5, C7, R7, U1, Y1

Commit message: esc changes
Parts:
- added C37: 1u, symbol Device:C
- added C38: 10n, symbol Device:C
- added C39, C40, C42: 100n, symbol Device:C
- added C41, C43: 47u, symbol Device:C
- added D10: SMBJ18A, SamacSys_Parts:SMBJ18A, symbol SamacSys_Parts:SMBJ18A
- added D11: LED, symbol Device:LED
- added FB3: 120R, symbol Device:FerriteBead
- added IC7: MA702GQ-P, QFN50P300X300X100-17N-D, symbol SamacSys_Parts:MA702GQ-P
- added L2: 22u, symbol Device:L
- added R29, R30, R31, R32, R33, R34: 10k, symbol Device:R
- added R35: 4k7, symbol Device:R
- added R36, R41: 1k, symbol Device:R
- added R37: 110k, symbol Device:R
- added R38: 12k, symbol Device:R
- added R39: 75k, symbol Device:R
- added R40: 24k, symbol Device:R
- added TP6841S7: ~, Package_TO_SOT_SMD:SOT-23-6, symbol New_Library:TP6841S6-A
Connections:
- net 3V3: now also C37.1, C43.1, D11.2 (A), IC7.13 (VDD), L2.2, R39.1
- net GND: now also C37.2, C38.2, C39.2, C40.2, C41.2, C43.2, D10.2 (A), IC7.10 (TEST), IC7.17 (GND_2), IC7.8 (GND_1), R29.2, R30.2, R31.1, R32.1, R33.1, R34.1, R36.2, R38.2, R40.2, R41.2, TP6841S7.2 (GND)
- net VCC_SENSE: now also C38.1, R35.2, R36.1
- net VISENSE_A: now also U1.14 (PA2); no longer U1.12 (PA0)
- net VISENSE_B: now also U1.12 (PA0); no longer U1.14 (PA2)
- net I2C_SCA: no longer names the net of U1.41 (PC9)
- net I2C_SCL: no longer names the net of U1.40 (PC8)
- new net: IC7.3 (Z), R31.2
- new net: IC7.1 (SSD), R29.1
- new net: IC7.15 (SSCK), R34.2
- new net: IC7.2 (A), R30.1
- new net: IC7.6 (B), R32.2
- new net: IC7.9 (PWM), R33.2
- new net BUCK_BST: C42.1, TP6841S7.1 (BST)
- new net BUCK_EN: R37.2, R38.1, TP6841S7.4 (EN)
- new net BUCK_FB: R39.2, R40.1, TP6841S7.3 (FB)
- new net BUCK_SW: C42.2, L2.1, TP6841S7.6 (SW)
- new net BUCK_VIN: C40.1, C41.1, FB3.2, R37.1, TP6841S7.5 (VIN)
- new net LED_PWR_K: D11.1 (K), R41.1
- new net MGH: IC7.16 (MGH)
- new net MGL: IC7.11 (MGL)
- new net SPI1_MISO: IC7.7 (MISO)
- new net SPI1_MOSI: IC7.4 (MOSI)
- new net SPI1_NSS: IC7.5 (CS)
- new net SPI1_SCK: IC7.12 (SCLK)
- new net VCC: C39.1, D10.1 (K), FB3.1, R35.1
- no-connect marks 0 -> 1
Other:
- sheet Phase renamed Phase_A
- removed sheet Power
- added sheet Phase_B (phase.kicad_sch)
- added sheet Phase_C (phase.kicad_sch)
- note added: "EXTERNAL CLOCK"
- note added: "MAGNETIC SENSOR"
- note added: "MCU"
- note added: "MOTOR PHASES"
- note added: "POWER SUPPLY"
- note added: "V_EN = 1.2V Vcc_low = 10.8V"
- moved on the sheet: C1, C15, C16, C17, C18, C19, C2, C3, C4, C5, C7, C8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

Commit message: full layout
Parts:
- removed D10: SMBJ18A, SamacSys_Parts:SMBJ18A, symbol SamacSys_Parts:SMBJ18A
- removed FB2, FB3: 120R, symbol Device:FerriteBead
- removed IC7: MA702GQ-P, QFN50P300X300X100-17N-D, symbol SamacSys_Parts:MA702GQ-P
- removed L2: 22u, symbol Device:L
- added B0-RST1: SW_Push, Button_Switch_SMD:SW_SPST_B3U-1000P, symbol Switch:SW_Push
- added C17, C18, C56, C58: 100n, Capacitor_SMD:C_0402_1005Metric, symbol Device:C
- added C19, C57: 1u, Capacitor_SMD:C_0603_1608Metric, symbol Device:C
- added D2: SMBJ18A, SamacSys_Parts:DIOM5436X244N, symbol SamacSys_Parts:SMBJ18A
- added FB1, FB2: MMZ1005F181ETD25, SamacSys_Parts:BEADC1005X55N, symbol SamacSys_Parts:MMZ1005F181ETD25
- added H1, H2, H3, H4: MountingHole, MountingHole:MountingHole_3.2mm_M3, symbol Mechanical:MountingHole
- added IC1: MA702GQ-P, SamacSys_Parts:QFN50P300X300X100-17N-D, symbol SamacSys_Parts:MA702GQ-P
- added J1: Conn_A, Connector_Wire:SolderWire-2sqmm_1x01_D2mm_OD3.9mm, symbol Connector:Conn_01x01_Socket
- added J2: Conn_B, Connector_Wire:SolderWire-2sqmm_1x01_D2mm_OD3.9mm, symbol Connector:Conn_01x01_Socket
- added J3: Conn_C, Connector_Wire:SolderWire-2sqmm_1x01_D2mm_OD3.9mm, symbol Connector:Conn_01x01_Socket
- added J4: KLDHCX-0202-BC-1, SamacSys_Parts:KLDHCX0202BC1, symbol SamacSys_Parts:KLDHCX-0202-BC-1
- added J5: USB_C_Receptacle_USB2.0_14P, Connector_USB:USB_C_Receptacle_Amphenol_12401610E4-2A, symbol Connector:USB_C_Receptacle_USB2.0_14P
- added J6: SWD_TagConnect_TC2030-NL, Connector:Tag-Connect_TC2030-IDC-NL_2x03_P1.27mm_Vertical, symbol Connector:Conn_ARM_SWD_TagConnect_TC2030-NL
- added L2: PA4343.682ANLT, SamacSys_Parts:INDPM135126X650N, symbol SamacSys_Parts:PA4343.682ANLT
- added R15, R16: 5k1, Resistor_SMD:R_0603_1608Metric, symbol Device:R
- added R19: 10k, Resistor_SMD:R_0603_1608Metric, symbol Device:R
- added U2: USBLC6-2SC6, Package_TO_SOT_SMD:SOT-23-6, symbol Power_Protection:USBLC6-2SC6
- C1: renamed from C42; footprint (none) -> Capacitor_SMD:C_0402_1005Metric; Link (none) -> https://www.mouser.de/ProductDetail/Murata-Electronics/GRM0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; MF (none) -> Murata Electronics; MP (none) -> GRM02YR60G104ME01L; MPN (none) -> 81-GRM02YR60G104ME1L
- C10: renamed from C3; footprint (none) -> Capacitor_SMD:C_0402_1005Metric; Link (none) -> https://www.mouser.de/ProductDetail/Murata-Electronics/GRM0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; MF (none) -> Murata Electronics; MP (none) -> GRM02YR60G104ME01L; MPN (none) -> 81-GRM02YR60G104ME1L
- C11: renamed from C4; footprint (none) -> Capacitor_SMD:C_0402_1005Metric; Link (none) -> https://www.mouser.de/ProductDetail/Murata-Electronics/GRM0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; MF (none) -> Murata Electronics; MP (none) -> GRM02YR60G104ME01L; MPN (none) -> 81-GRM02YR60G104ME1L
- C12: renamed from C5; footprint (none) -> Capacitor_SMD:C_0402_1005Metric; Link (none) -> https://www.mouser.de/ProductDetail/Murata-Electronics/GRM0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; MF (none) -> Murata Electronics; MP (none) -> GRM02YR60G104ME01L; MPN (none) -> 81-GRM02YR60G104ME1L
- C13: renamed from C37; footprint (none) -> Capacitor_SMD:C_0603_1608Metric; Link (none) -> https://www.mouser.de/ProductDetail/TAIYO-YUDEN/MBJCT168CB7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; MF (none) -> TAIYO YUDEN; MP (none) -> MBJCT168CB7105KRPA01; MPN (none) -> 963-BJCT168CB7105KR
- C14: renamed from C19; footprint (none) -> Capacitor_SMD:C_0402_1005Metric; Link (none) -> https://www.mouser.de/ProductDetail/Murata-Electronics/GRM0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; MF (none) -> Murata Electronics; MP (none) -> GRM02YR60G104ME01L; MPN (none) -> 81-GRM02YR60G104ME1L
- C15: renamed from C8; footprint (none) -> Capacitor_SMD:C_0402_1005Metric; Link (none) -> https://www.mouser.de/ProductDetail/Murata-Electronics/GRM0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; MF (none) -> Murata Electronics; MP (none) -> GRM02YR60G104ME01L; MPN (none) -> 81-GRM02YR60G104ME1L
- C16: renamed from C18; footprint (none) -> Capacitor_SMD:C_0402_1005Metric; Link (none) -> https://www.mouser.de/ProductDetail/Murata-Electronics/GRM0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; MF (none) -> Murata Electronics; MP (none) -> GRM02YR60G104ME01L; MPN (none) -> 81-GRM02YR60G104ME1L
- C2: renamed from C43; footprint (none) -> Capacitor_SMD:C_1206_3216Metric; Link (none) -> https://www.mouser.de/ProductDetail/TDK/C3216X5R1E476M160AC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; MF (none) -> TDK; MP (none) -> C3216X5R1E476M160AC; MPN (none) -> 810-C3216X5R1E476M; Manufacturer_Part_Number (none) -> MLASE31LBB5476MTNA01; Mouser Part Number (none) -> 963-MLASE31LBB5476MT
- C20: renamed from C15; footprint (none) -> Capacitor_SMD:C_0402_1005Metric; Link (none) -> https://www.mouser.de/ProductDetail/Murata-Electronics/GRM0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; MF (none) -> Murata Electronics; MP (none) -> GRM02YR60G104ME01L; MPN (none) -> 81-GRM02YR60G104ME1L
- C21: renamed from C17; footprint (none) -> Capacitor_SMD:C_0402_1005Metric; Link (none) -> https://www.mouser.de/ProductDetail/Murata-Electronics/GJM0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; MF (none) -> Murata Electronics; MP (none) -> GJM0225C1C6R8CB01L; MPN (none) -> 81-GJM0225C1C6R8CB1L
- C22: renamed from C16; footprint (none) -> Capacitor_SMD:C_0402_1005Metric; Link (none) -> https://www.mouser.de/ProductDetail/Murata-Electronics/GJM0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; MF (none) -> Murata Electronics; MP (none) -> GJM0225C1C6R8CB01L; MPN (none) -> 81-GJM0225C1C6R8CB1L
- C3: renamed from C39; footprint (none) -> Capacitor_SMD:C_0402_1005Metric; Link (none) -> https://www.mouser.de/ProductDetail/Murata-Electronics/GRM0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; MF (none) -> Murata Electronics; MP (none) -> GRM02YR60G104ME01L; MPN (none) -> 81-GRM02YR60G104ME1L
- C4: renamed from C40; footprint (none) -> Capacitor_SMD:C_0402_1005Metric; Link (none) -> https://www.mouser.de/ProductDetail/Murata-Electronics/GRM0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; MF (none) -> Murata Electronics; MP (none) -> GRM02YR60G104ME01L; MPN (none) -> 81-GRM02YR60G104ME1L
- C5: renamed from C41; footprint (none) -> Capacitor_SMD:C_1206_3216Metric; Link (none) -> https://www.mouser.de/ProductDetail/TDK/C3216X5R1E476M160AC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; MF (none) -> TDK; MP (none) -> C3216X5R1E476M160AC; MPN (none) -> 810-C3216X5R1E476M; Manufacturer_Part_Number (none) -> MLASE31LBB5476MTNA01; Mouser Part Number (none) -> 963-MLASE31LBB5476MT
- C6: renamed from C38; footprint (none) -> Capacitor_SMD:C_0402_1005Metric; Link (none) -> https://www.mouser.de/ProductDetail/Vishay-Vitramon/VJ0402Y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; MF (none) -> Vishay / Vitramon; MP (none) -> VJ0402Y103KXJAC31X; MPN (none) -> 77-V0402Y103KXJAC31X
- C7: footprint (none) -> Capacitor_SMD:C_0603_1608Metric; Link (none) -> https://www.mouser.de/ProductDetail/TAIYO-YUDEN/MLASE168AB5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; MF (none) -> TAIYO YUDEN; MP (none) -> MLASE168AB5475KTNA01; MPN (none) -> 963-MLASE168AB5475KT
- C8: renamed from C1; footprint (none) -> Capacitor_SMD:C_0402_1005Metric; Link (none) -> https://www.mouser.de/ProductDetail/Murata-Electronics/GRM0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; MF (none) -> Murata Electronics; MP (none) -> GRM02YR60G104ME01L; MPN (none) -> 81-GRM02YR60G104ME1L
- C9: renamed from C2; footprint (none) -> Capacitor_SMD:C_0402_1005Metric; Link (none) -> https://www.mouser.de/ProductDetail/Murata-Electronics/GRM0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; MF (none) -> Murata Electronics; MP (none) -> GRM02YR60G104ME01L; MPN (none) -> 81-GRM02YR60G104ME1L
- D1: renamed from D11; footprint (none) -> LED_SMD:LED_0603_1608Metric; Link (none) -> https://www.mouser.de/ProductDetail/ams-OSRAM/GW-JTLMS3.GM-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; MF (none) -> ams OSRAM; MP (none) -> GW JTLMS3.GM-G3G7-XX58-1-60-R33; MPN (none) -> 720-GWJTLMS3.G3G758
- D3: footprint (none) -> LED_SMD:LED_0603_1608Metric; Link (none) -> https://www.mouser.de/ProductDetail/ams-OSRAM/GW-JTLMS3.GM-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; MF (none) -> ams OSRAM; MP (none) -> GW JTLMS3.GM-G3G7-XX58-1-60-R33; MPN (none) -> 720-GWJTLMS3.G3G758
- R1: renamed from R35; footprint (none) -> Resistor_SMD:R_0603_1608Metric; Link (none) -> https://www.mouser.de/ProductDetail/KOA-Speer/RN73H1ETTP470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; MF (none) -> KOA Speer; MP (none) -> RN73H1ETTP4701D25; MPN (none) -> 660-RN73H1ETP4701D25
- R10: renamed from R29; footprint (none) -> Resistor_SMD:R_0603_1608Metric; Link (none) -> https://www.mouser.de/ProductDetail/Panasonic/ERA-1AEB103C?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; MF (none) -> Panasonic; MP (none) -> ERA-1AEB103C; MPN (none) -> 667-ERA-1AEB103C
- R11: renamed from R30; footprint (none) -> Resistor_SMD:R_0603_1608Metric; Link (none) -> https://www.mouser.de/ProductDetail/Panasonic/ERA-1AEB103C?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; MF (none) -> Panasonic; MP (none) -> ERA-1AEB103C; MPN (none) -> 667-ERA-1AEB103C
- R12: renamed from R31; footprint (none) -> Resistor_SMD:R_0603_1608Metric; Link (none) -> https://www.mouser.de/ProductDetail/Panasonic/ERA-1AEB103C?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; MF (none) -> Panasonic; MP (none) -> ERA-1AEB103C; MPN (none) -> 667-ERA-1AEB103C
- R13: renamed from R33; footprint (none) -> Resistor_SMD:R_0603_1608Metric; Link (none) -> https://www.mouser.de/ProductDetail/Panasonic/ERA-1AEB103C?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; MF (none) -> Panasonic; MP (none) -> ERA-1AEB103C; MPN (none) -> 667-ERA-1AEB103C
- R14: renamed from R32; footprint (none) -> Resistor_SMD:R_0603_1608Metric; Link (none) -> https://www.mouser.de/ProductDetail/Panasonic/ERA-1AEB103C?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; MF (none) -> Panasonic; MP (none) -> ERA-1AEB103C; MPN (none) -> 667-ERA-1AEB103C
- R17: renamed from R10; value 10k -> 1k; footprint (none) -> Resistor_SMD:R_0603_1608Metric; Link (none) -> https://www.mouser.de/ProductDetail/Vishay-Dale/CRCW06031K0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; MF (none) -> Vishay / Dale; MP (none) -> CRCW06031K00FKED; MPN (none) -> 71-CRCW06031K00FKED
- R18: renamed from R7; value 10k -> 100R; footprint (none) -> Resistor_SMD:R_0603_1608Metric; Link (none) -> https://www.mouser.de/ProductDetail/Susumu/RG0603P-101-D-T1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; MF (none) -> Susumu; MP (none) -> RG0603P-101-D-T10; MPN (none) -> 754-RG0603P-101-D
- R2: renamed from R37; footprint (none) -> Resistor_SMD:R_0603_1608Metric; Link (none) -> https://www.mouser.de/ProductDetail/Vishay-Beyschlag/MCT060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; MF (none) -> Vishay / Beyschlag; MP (none) -> MCT06030C1103FP500; MPN (none) -> 594-MCT06030C1103FP5
- R3: renamed from R39; footprint (none) -> Resistor_SMD:R_0603_1608Metric; Link (none) -> https://www.mouser.de/ProductDetail/YAGEO/RT0603FRE1375KL?q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; MF (none) -> YAGEO; MP (none) -> RT0603FRE1375KL; MPN (none) -> 603-RT0603FRE1375KL
- R4: renamed from R41; footprint (none) -> Resistor_SMD:R_0603_1608Metric; Link (none) -> https://www.mouser.de/ProductDetail/Vishay-Dale/CRCW06031K0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; MF (none) -> Vishay / Dale; MP (none) -> CRCW06031K00FKED; MPN (none) -> 71-CRCW06031K00FKED
- R5: renamed from R38; footprint (none) -> Resistor_SMD:R_0603_1608Metric; Link (none) -> https://www.mouser.de/ProductDetail/Vishay-Beyschlag/MCS040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; MF (none) -> Vishay / Beyschlag; MP (none) -> MCS04020D1202BE000; MPN (none) -> 594-MCS04020D1202BE0
- R6: renamed from R36; footprint (none) -> Resistor_SMD:R_0603_1608Metric; Link (none) -> https://www.mouser.de/ProductDetail/Vishay-Dale/CRCW06031K0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; MF (none) -> Vishay / Dale; MP (none) -> CRCW06031K00FKED; MPN (none) -> 71-CRCW06031K00FKED
- R7: renamed from R40; footprint (none) -> Resistor_SMD:R_0603_1608Metric; Link (none) -> https://www.mouser.de/ProductDetail/Panasonic/ERA-3AEB243V?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; MF (none) -> Panasonic; MP (none) -> ERA-3AEB243V; MPN (none) -> 667-ERA-3AEB243V
- R8: renamed from R34; footprint (none) -> Resistor_SMD:R_0603_1608Metric; Link (none) -> https://www.mouser.de/ProductDetail/Panasonic/ERA-1AEB103C?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; MF (none) -> Panasonic; MP (none) -> ERA-1AEB103C; MPN (none) -> 667-ERA-1AEB103C
- R9: footprint (none) -> Resistor_SMD:R_0603_1608Metric; Link (none) -> https://www.mouser.de/ProductDetail/Panasonic/ERA-1AEB103C?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; MF (none) -> Panasonic; MP (none) -> ERA-1AEB103C; MPN (none) -> 667-ERA-1AEB103C
- TP6841S1: renamed from TP6841S7; Link (none) -> https://lcsc.com/product-detail/DC-DC-Converters_TECH-PUBLI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; MF (none) -> TECH PUBLIC; MP (none) -> TP6841S6-A
Connections:
- net 3V3: now also C16.1, R18.1, C58.1, FB2.2, IC1.13 (VDD), J6.1 (VCC), L2.2; no longer C15.1, R18.2, U1.28 (VREF+), U1.29 (VDDA)
- net BUCK_SW: now also L2.1
- net BUCK_VIN: now also FB1.2
- net GND: now also C17.2, C18.2, C19.2, C56.2, C57.2, C58.2, D2.1 (K), IC1.10 (TEST), IC1.17 (GND_2), IC1.8 (GND_1), J4.2, J5.A1 (GND), J5.A12 (GND), J5.B1 (GND), J5.B12 (GND), J5.S1 (SHIELD), J6.5 (GND), R15.2, R16.2, R19.2, U2.2 (GND)
- net HIN_A: now also U1.38 (PC6); no longer U1.42 (PA8)
- net HIN_B: now also U1.36 (PB14); no longer U1.43 (PA9)
- net HIN_C: now also U1.34 (PB12); no longer U1.44 (PA10)
- net LIN_A: now also U1.39 (PC7)
- net LIN_B: now also U1.37 (PB15)
- net LIN_C: now also U1.35 (PB13)
- net VCC: now also D2.2 (A), FB1.1, J4.1
- net VISENSE_A: now also U1.12 (PA0); no longer U1.14 (PA2)
- net VISENSE_B: now also U1.13 (PA1); no longer U1.12 (PA0)
- net VISENSE_C: now also U1.14 (PA2); no longer U1.10 (PC2)
- net VPH_A: now also J1.1 (Pin_1)
- net VPH_B: now also J2.1 (Pin_1)
- net VPH_C: now also J3.1 (Pin_1)
- net VSENSE_A: now also U1.9 (PC1)
- net VSENSE_B: now also U1.10 (PC2)
- net VSENSE_C: now also U1.11 (PC3)
- net LED_MCU: now reaches D3.2 (A), U1.2 (PC13)
- net MG_Z: now reaches R12.2
- net MG_Z: now also IC1.3 (Z)
- net MCU_NRST: now reaches C14.1, R9.1, U1.7 (PG10)
- net MCU_NRST: now also J6.3 (~{RESET})
- net SSD: now reaches R10.1
- net SSD: now also IC1.1 (SSD)
- net SSCK: now reaches R8.2
- net SSCK: now also IC1.15 (SSCK)
- net MG_A: now reaches R11.1
- net MG_A: now also IC1.2 (A)
- net MG_B: now reaches R14.2
- net MG_B: now also IC1.6 (B)
- net MG_PWM: now reaches R13.2
- net MG_PWM: now also IC1.9 (PWM)
- net BOOT0: now reaches C20.1, U1.61 (PB8)
- net BOOT0: now also B0-RST1.1, R19.1; no longer R18.1
- net SG_1: now reaches U1.17 (PA3)
- net MGH_SPI1_NSS: now reaches U1.18 (PA4)
- net MGH_SPI1_NSS: now also IC1.5 (CS)
- net MGH_SPI1_SCK: now reaches U1.19 (PA5)
- net MGH_SPI1_SCK: now also IC1.12 (SCLK)
- net MGH_SPI1_MISO: now reaches U1.20 (PA6)
- net MGH_SPI1_MISO: now also IC1.7 (MISO)
- net MGH_SPI1_MOSI: now reaches U1.21 (PA7)
- net MGH_SPI1_MOSI: now also IC1.4 (MOSI)
- net SG_2: now reaches U1.22 (PC4)
- net SG_3: now reaches U1.23 (PC5)
- net MGH_MGH: now reaches U1.24 (PB0)
- net MGH_MGH: now also IC1.16 (MGH)
- net MGH_MGL: now reaches U1.25 (PB1)
- net MGH_MGL: now also IC1.11 (MGL)
- net USB_D-: now reaches U1.45 (PA11)
- net USB_D-: now also C18.1, U2.6 (I/O1)
- net USB_D+: now reaches U1.46 (PA12)
- net USB_D+: now also C17.1, U2.4 (I/O2)
- net MCU_SWDIO: now reaches U1.49 (PA13)
- net MCU_SWDIO: now also J6.2 (SWDIO)
- net MCU_SWCLK: now reaches U1.50 (PA14)
- net MCU_SWCLK: now also J6.4 (SWCLK)
- net MCU_SWO: now reaches U1.56 (PB3)
- net MCU_SWO: now also J6.6 (SWO)
- new net: B0-RST1.2, R18.2
- new net 3V3_Filt: C15.1, C56.1, C57.1, FB2.1, U1.28 (VREF+), U1.29 (VDDA)
- new net USB_AB+: J5.A6 (D+), J5.B6 (D+), U2.3 (I/O2)
- new net USB_AB-: J5.A7 (D-), J5.B7 (D-), U2.1 (I/O1)
- new net USB_DBCC1: J5.B5 (CC2), R15.1, U1.44 (PA10)
- new net USB_DBCC2: J5.A5 (CC1), R16.1, U1.43 (PA9)
- new net VBUS: C19.1, J5.A4 (VBUS), J5.A9 (VBUS), J5.B4 (VBUS), J5.B9 (VBUS), U2.5 (VBUS)
- no-connect marks 1 -> 20
Other:
- added sheet Amplifier (amplify.kicad_sch)
- added sheet Amplifier1 (amplify.kicad_sch)
- added sheet Amplifier2 (amplify.kicad_sch)
- note added: "AMPLIFIERS FORCE"
- note added: "CONNECTORS"
- note added: "Power Connector"
- note added: "TAG SWD Connector"
- note added: "USBC Connection"
- moved on the sheet: C10, C11, C12, C13, C15, C16, C2, C20, C21, C22, C7, C8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

Commit message: ready for production..?
Parts:
- removed J5: USB_C_Receptacle_USB2.0_14P, Connector_USB:USB_C_Receptacle_Amphenol_12401610E4-2A, symbol Connector:USB_C_Receptacle_USB2.0_14P
- added J7: USB4510-03-1-A, USB4510031A, symbol SamacSys_Parts:USB4510-03-1-A
- J4: Link (none) -> https://www.mouser.de/ProductDetail/Kycon/KLDHCX-0202-BC-1?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; MF (none) -> Kycon; MP (none) -> KLDHCX-0202-BC-1; MPN (none) -> 806-KLDHCX-0202-BC-1
- U1: Link (none) -> https://www.mouser.de/ProductDetail/STMicroelectronics/STM3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; MF (none) -> STMicroelectronics; MP (none) -> STM32G474RET6; MPN (none) -> 511-STM32G474RET6
- U2: Link (none) -> https://www.mouser.de/ProductDetail/STMicroelectronics/USBL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; MF (none) -> STMicroelectronics; MP (none) -> USBLC6-2SC6; MPN (none) -> 511-USBLC6-2SC6
- Y1: Link (none) -> https://www.mouser.de/ProductDetail/NDK/NX2016SA-24M-EXS00A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; MF (none) -> NDK; MP (none) -> NX2016SA-24M-EXS00A-CS08891; MPN (none) -> 344-NX2016SA24S08891
Connections:
- net GND: now also J7.A1 (GND_1), J7.A12 (GND_2), J7.MH1, J7.MH2, J7.MH3, J7.MH4
- net USB_AB+: now also J7.A6 (DP1), J7.B6 (DP2)
- net USB_AB-: now also J7.A7 (DN1), J7.B7 (DN2)
- net USB_DBCC1: now also R16.1, J7.A5 (CC1); no longer R15.1
- net USB_DBCC2: now also R15.1, J7.B5 (CC2); no longer R16.1
- net VBUS: now also J7.A4 (VBUS_1), J7.A9 (VBUS_2)
- no-connect marks 20 -> 22
Other:
- moved on the sheet: C19, C21, C22, C58, H1, H2, H3, H4, J4, J6, R15, R16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

Commit message: adding esc kicad and stm32cubeide project
Parts:
- added J5: Conn_01x06_Socket, Connector_PinSocket_2.54mm:PinSocket_1x06_P2.54mm_Vertical, symbol Connector:Conn_01x06_Socket
- D2: value SMBJ18A -> SMBJ188A
- J1, J2, J3: Link (none) -> will not be populated and soldered by customer; MF (none) -> -; MP (none) -> -; MPN (none) -> -
- J7: footprint USB4510031A -> SamacSys_Parts:USB4510031A
- R1: Link https://www.mouser.de/ProductDetail/KOA-Speer/RN73H1ETTP470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 -> https://www.mouser.de/ProductDetail/Susumu/RG1608N-472-W-T5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; MF KOA Speer -> Susumu; MP RN73H1ETTP4701D25 -> RG1608N-472-W-T5; MPN 660-RN73H1ETP4701D25 -> 754-RG1608N-472-WT5
- R10, R11, R12, R13, R14, R19, R8, R9: Link https://www.mouser.de/ProductDetail/Panasonic/ERA-1AEB103C?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 -> https://www.mouser.de/ProductDetail/SEI-Stackpole/RNCE0603B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; MF Panasonic -> SEI Stackpole; MP ERA-1AEB103C -> RNCE0603BTE10K0; MPN 667-ERA-1AEB103C -> 708-RNCE0603BTE10K0
- R15, R16: Link https://www.mouser.de/ProductDetail/Panasonic/ERA-1AEB512C?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 -> https://www.mouser.de/ProductDetail/Vishay-Beyschlag/MCT060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; MF Panasonic -> Vishay / Beyschlag; MP ERA-1AEB512C -> MCT06030C5101FPW00; MPN 667-ERA-1AEB512C -> 594-MCT06030C5101FPW
- R18: Link https://www.mouser.de/ProductDetail/Susumu/RG0603P-101-D-T1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 -> https://www.mouser.de/ProductDetail/SEI-Stackpole/RNCE0603B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; MF Susumu -> SEI Stackpole; MP RG0603P-101-D-T10 -> RNCE0603BTE100R; MPN 754-RG0603P-101-D -> 708-RNCE0603BTE100R
- Y1: value NX2016SA-24M-EXS00A-CS08891 -> CS08891-24M; MP NX2016SA-24M-EXS00A-CS08891 -> CS08891-24M
Connections:
- net 3V3: now also J5.2 (Pin_2)
- net GND: now also J5.3 (Pin_3)
- net RXD: now reaches U1.54 (PC12)
- net RXD: now also J5.5 (Pin_5)
- net TXD: now reaches U1.55 (PD2)
- net TXD: now also J5.4 (Pin_4)
Other:
- note added: "Bluetooth header UART"

Commit message: with the used libraries
Connections:
- net GND: now also D2.2 (A); no longer D2.1 (K)
- net VCC: now also D2.1 (K); no longer D2.2 (A)
Other:
- moved on the sheet: D2
Changed lines of the file:
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@@
 	(symbol
 		(lib_id "SamacSys_Parts:SMBJ18A")
-		(at 34.29 62.23 90)
+		(at 34.29 46.99 270)
 		(unit 1)
 		(exclude_from_sim no)
@@
 		(fields_autoplaced yes)
 		(property "Reference" "D2"
-			(at 38.1 53.8479 90)
+			(at 38.1 52.8319 90)
 			(effects
 				(font
 					(size 1.27 1.27)
 				)
-				(justify right)
+				(justify left)
 			)
 		)
 		(property "Value" "SMBJ188A"
-			(at 38.1 56.3879 90)
+			(at 38.1 55.3719 90)
 			(effects
 				(font
 					(size 1.27 1.27)
 				)
-				(justify right)
+				(justify left)
 			)
 		)
 		(property "Footprint" "SamacSys_Parts:DIOM5436X244N"
-			(at 127.94 52.07 0)
+			(at -59.36 57.15 0)
 			(effects
 				(font
@@
 		)
 		(property "Datasheet" "http://www.vishay.com/docs/88392/smbj.pdf"
-			(at 227.94 52.07 0)
+			(at -159.36 57.15 0)
 			(effects
 				(font
@@
 		)
 		(property "Description" "SMBJ18A"
-			(at 34.29 62.23 0)
+			(at 34.29 46.99 0)
 			(effects
 				(font
@@
 		)
 		(property "Height" "2.44"
-			(at 427.94 52.07 0)
+			(at -359.36 57.15 0)
 			(effects
 				(font
@@
 		)
 		(property "Manufacturer_Name" "Vishay"
-			(at 527.94 52.07 0)
+			(at -459.36 57.15 0)
 			(effects
 				(font
@@
 		)
 		(property "Manufacturer_Part_Number" "SMBJ18A"
-			(at 627.94 52.07 0)
+			(at -559.36 57.15 0)
 			(effects
 				(font
@@
 		)
 		(property "Mouser Part Number" ""
-			(at 727.94 52.07 0)
+			(at -659.36 57.15 0)
 			(effects
 				(font
@@
 		)
 		(property "Mouser Price/Stock" ""
-			(at 827.94 52.07 0)
+			(at -759.36 57.15 0)
 			(effects
 				(font
@@
 		)
 		(property "Arrow Part Number" ""
-			(at 927.94 52.07 0)
+			(at -859.36 57.15 0)
 			(effects
 				(font
@@
 		)
 		(property "Arrow Price/Stock" ""
-			(at 1027.94 52.07 0)
+			(at -959.36 57.15 0)
 			(effects
 				(font
@@
 		)
 		(property "Link" "https://www.mouser.de/ProductDetail/Littelfuse/SMBJ188A?qs=zHiv0nsVGmqpK5qihuf5vg%3D%3D"
-			(at 34.29 62.23 0)
+			(at 34.29 46.99 0)
 			(effects
 				(font
@@
 		)
 		(property "MF" " Littelfuse "
-			(at 34.29 62.23 0)
+			(at 34.29 46.99 0)
 			(effects
 				(font
@@
 		)
 		(property "MP" "SMBJ188A "
-			(at 34.29 62.23 0)
+			(at 34.29 46.99 0)
 			(effects
 				(font
@@
 		)
 		(property "MPN" "576-SMBJ188A "
-			(at 34.29 62.23 0)
+			(at 34.29 46.99 0)
 			(effects
 				(font
